Commit message: feat: fk calc (#2)
- Implemented compute_fk method to compute forward kinematics.
- Using k library to cross-check compute_fk method with k output (assuming k is ground truth).

File: assets/simple_robot.urdf (robot description, URDF)
Before this commit: robot simple_arm, 4 links, 3 joints
Links:
- removed link elbow_link
- removed link shoulder_link
- removed link wrist_link
- added link forearm; visual cylinder length=0.8 radius=0.04
- added link upper_arm; visual cylinder length=1.0 radius=0.05
- link base_link: geometry visual cylinder length=0.1 radius=0.2
Joints:
- removed joint wrist_joint
- joint elbow_joint: child elbow_link -> forearm; limit lower=-1.57 upper=1.57 effort=10 velocity=1.0 -> lower=-1.57 upper=1.57 effort=100.0 velocity=1.0; origin xyz=0 0 0.3 rpy=0 0 0 -> xyz=0 0 0.9 rpy=0 0 0; parent shoulder_link -> upper_arm
- joint shoulder_joint: child shoulder_link -> upper_arm; limit lower=-1.57 upper=1.57 effort=10 velocity=1.0 -> lower=-1.57 upper=1.57 effort=100.0 velocity=1.0
